Commit message: finish jaco urdf

File: ada_description/robots/jaco.urdf (robot description, URDF)
Before this commit: robot ADA, 16 links, 15 joints
Links:
- removed link mico_link_finger_3
- removed link mico_link_finger_tip_3
Joints:
- removed joint mico_joint_finger_3
- removed joint mico_joint_finger_tip_3
- joint mico_joint_2: limit lower=0.820304748437 upper=5.46288055874 effort=2000 velocity=1 -> lower=-3.83 upper=0.784 effort=2000 velocity=1
- joint mico_joint_3: limit lower=0.331612557879 upper=5.9515727493 effort=2000 velocity=1 -> lower=-4.38805378 upper=1.233854435 effort=2000 velocity=1
